File: EP-Booster/EP-Booster.kicad_pcb (KiCad board)
At the start: 2 copper layers, 52.5 x 85.5 mm, 37 parts, among them Q1 MMBF5457_, Q2 BC849, SW1 SW_DIP_x02

Commit message: Revision 1
Parts:
- moved R12 0.50 mm to (147.5, 81.6)
- moved R2 0.50 mm to (147.6, 84.4)
Routing:
- net Net-(C7-Pad2): track 29.3 -> 24.3 mm
- net /VB: track 15.2 -> 15.7 mm
- net /SWA2: track 45.0 -> 44.5 mm
Changed lines of the file:
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@@
 		(48 "B.Fab" user)
 		(49 "F.Fab" user)
-		(50 "User.1" user)
-		(51 "User.2" user)
-		(52 "User.3" user)
-		(53 "User.4" user)
-		(54 "User.5" user)
-		(55 "User.6" user)
-		(56 "User.7" user)
-		(57 "User.8" user)
-		(58 "User.9" user)
 	)
 	(setup
+		(stackup
+			(layer "F.SilkS"
+				(type "Top Silk Screen")
+			)
+			(layer "F.Paste"
+				(type "Top Solder Paste")
+			)
+			(layer "F.Mask"
+				(type "Top Solder Mask")
+				(thickness 0.01)
+			)
+			(layer "F.Cu"
+				(type "copper")
+				(thickness 0.035)
+			)
+			(layer "dielectric 1"
+				(type "core")
+				(thickness 1.51)
+				(material "FR4")
+				(epsilon_r 4.5)
+				(loss_tangent 0.02)
+			)
+			(layer "B.Cu"
+				(type "copper")
+				(thickness 0.035)
+			)
+			(layer "B.Mask"
+				(type "Bottom Solder Mask")
+				(thickness 0.01)
+			)
+			(layer "B.Paste"
+				(type "Bottom Solder Paste")
+			)
+			(layer "B.SilkS"
+				(type "Bottom Silk Screen")
+			)
+			(copper_finish "None")
+			(dielectric_constraints no)
+		)
 		(pad_to_mask_clearance 0)
 		(allow_soldermask_bridges_in_footprints no)
@@
 	(footprint "Library:StandardResistorPedal"
 		(layer "F.Cu")
-		(at 147.1 84.36 -90)
+		(at 147.6 84.41 -90)
 		(descr "Resistor, Axial_DIN0207 series, Axial, Horizontal, pin pitch=7.62mm, 0.25W = 1/4W, length*diameter=6.3*2.5mm^2, http://cdn-reichelt.de/documents/datenblatt/B400/1_4W%23YAG.pdf")
 		(tags "Resistor Axial_DIN0207 series Axial Horizontal pin pitch 7.62mm 0.25W = 1/4W length 6.3mm diameter 2.5mm")
@@
 	(footprint "Library:StandardResistorPedal"
 		(layer "F.Cu")
-		(at 147 81.51 90)
+		(at 147.5 81.56 90)
 		(descr "Resistor, Axial_DIN0207 series, Axial, Horizontal, pin pitch=7.62mm, 0.25W = 1/4W, length*diameter=6.3*2.5mm^2, http://cdn-reichelt.de/documents/datenblatt/B400/1_4W%23YAG.pdf")
 		(tags "Resistor Axial_DIN0207 series Axial Horizontal pin pitch 7.62mm 0.25W = 1/4W length 6.3mm diameter 2.5mm")
 		(property "Reference" "R12"
-			(at 4.01 -2 90)
+			(at 4.01 -2.25 90)
 			(layer "F.SilkS")
 			(effects
@@
 		(tags "Resistor Axial_DIN0207 series Axial Horizontal pin pitch 7.62mm 0.25W = 1/4W length 6.3mm diameter 2.5mm")
 		(property "Reference" "R3"
-			(at 3.81 -2.37 0)
+			(at 3.28 -2.294888 0)
 			(layer "F.SilkS")
 			(effects
@@
 	)
 	(segment
-		(start 146.055112 81.51)
-		(end 147 81.51)
+		(start 144.734888 78.794888)
+		(end 147.5 81.56)
 		(width 0.2)
 		(layer "F.Cu")
@@
 	(segment
 		(start 143.34 78.794888)
-		(end 146.055112 81.51)
+		(end 144.734888 78.794888)
 		(width 0.2)
 		(layer "F.Cu")
@@
 	)
 	(segment
-		(start 148.19 73.89)
-		(end 152.5 78.2)
-		(width 0.2)
-		(layer "F.Cu")
-		(net 8)
-	)
-	(segment
 		(start 155.4 83.171068)
 		(end 155.4 87.578932)
@@
 	)
 	(segment
-		(start 147 73.89)
-		(end 148.19 73.89)
+		(start 152.5 78.2)
+		(end 148.24 73.94)
+		(width 0.2)
+		(layer "F.Cu")
+		(net 8)
+	)
+	(segment
+		(start 148.24 73.94)
+		(end 147.5 73.94)
 		(width 0.2)
 		(layer "F.Cu")
@@
 	)
 	(segment
-		(start 148.5 43.05)
-		(end 146.7 41.25)
+		(start 130.201068 41)
+		(end 139.378932 41)
+		(width 0.2)
+		(layer "F.Cu")
+		(net 11)
+	)
+	(segment
+		(start 125.63 43.5)
+		(end 126.665534 42.464466)
 		(width 0.2)
 		(layer "F.Cu")
@@
 	)
 	(segment
-		(start 146.7 41.25)
-		(end 129.951068 41.25)
+		(start 142.914466 42.464466)
+		(end 143.5 43.05)
 		(width 0.2)
 		(layer "F.Cu")
 		(net 11)
 	)
-	(segment
-		(start 126.415534 42.714466)
-		(end 125.63 43.5)
+	(arc
+		(start 130.201068 41)
+		(mid 128.287651 41.380602)
+		(end 126.665534 42.464466)
 		(width 0.2)
 		(layer "F.Cu")
@@
 	)
 	(arc
-		(start 126.415534 42.714466)
-		(mid 128.037651 41.630602)
-		(end 129.951068 41.25)
+		(start 142.914466 42.464466)
+		(mid 141.292349 41.380602)
+		(end 139.378932 41)
 		(width 0.2)
 		(layer "F.Cu")

Commit message: V2.0
Parts:
- added H10: MountingHole_Pad, MountingHole:MountingHole_2.2mm_M2_DIN965_Pad, F.Cu at (162.2, 27.0)
- added H11: MountingHole_Pad, MountingHole:MountingHole_2.2mm_M2_DIN965_Pad, F.Cu at (123.8, 88.8)
- added H12: MountingHole_Pad, MountingHole:MountingHole_2.2mm_M2_DIN965_Pad, F.Cu at (162.2, 88.8)
- added H9: MountingHole_Pad, MountingHole:MountingHole_2.2mm_M2_DIN965_Pad, F.Cu at (123.8, 27.0)
- C5: value 33n -> 10u
- R14: value 100R -> 100
- R2: value 390R -> 390
- moved R15 29.9 mm to (161.8, 54.8)
- moved R14 25.8 mm to (154.2, 50.5), turned to 0 degrees
- moved H1 22.8 mm to (151.2, 97.0), turned to 0 degrees
- moved R16 18.7 mm to (157.0, 62.3)
- moved SW1 18.7 mm to (158.2, 73.3)
- moved D1 15.7 mm to (138.2, 88.2), turned to 0 degrees
- moved RV1 15.6 mm to (138.0, 31.5), turned to 90 degrees
- moved H2 15.1 mm to (126.0, 97.0)
- moved H8 15.0 mm to (146.1, 97.0)
- moved R13 14.6 mm to (162.0, 39.9)
- moved C6 14.4 mm to (158.0, 37.0), turned to 180 degrees
- moved H5 13.2 mm to (131.0, 97.0)
- moved H7 11.4 mm to (141.1, 97.0)
- moved H4 11.2 mm to (156.2, 97.0)
- moved H6 10.9 mm to (136.1, 97.0)
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Routing:
- net /SWB2: track 18.8 -> 46.0 mm
- net Net-(C3-Pad1): track 11.6 -> 36.4 mm
- net /SWA1: track 36.4 -> 17.9 mm
- net Net-(C6-Pad2): track 26.4 -> 14.0 mm
- net Net-(D2-K): track 5.73 -> 17.1 mm
- net /SWB1: track 13.4 -> 23.9 mm
- net Net-(C7-Pad2): track 24.3 -> 14.0 mm
- net Net-(D2-A): track 4.92 -> 13.8 mm
- net +9V: track 4.36 -> 11.8 mm
- net /SWA2: track 44.5 -> 37.8 mm
- net Net-(Q2-E): track 7.84 -> 14.1 mm
- net Net-(D1-K): track 12.6 -> 16.0 mm
- net Net-(C3-Pad2): track 7.28 -> 9.64 mm
- net Net-(C7-Pad1): track 14.6 -> 12.8 mm
- net Net-(Q1-Pad3): track 8.67 -> 10.2 mm
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Other:
- board size 52.5 x 85.5 mm -> 44.2 x 78.2 mm
