File: EP-Booster/EP-Booster.kicad_sch (KiCad schematic)
At the start: 29 parts, among them Q1 MMBF5457_, Q2 BC849, SW1 SW_DIP_x02

Commit message: first proto
Parts:
- added H1: SW., Library:1.5mm_MountingHole, symbol Mechanical:MountingHole_Pad
- added H2: IN, Library:1.5mm_MountingHole, symbol Mechanical:MountingHole_Pad
- added H3: OUT, Library:1.5mm_MountingHole, symbol Mechanical:MountingHole_Pad
- added H4, H5, H6, H8: Earth, Library:1.5mm_MountingHole, symbol Mechanical:MountingHole_Pad
- added H7: +9V, Library:1.5mm_MountingHole, symbol Mechanical:MountingHole_Pad
- C1, C2, C4, C6, C7: footprint (none) -> Library:StandardPolarizedCapacitorPedal
- C3, C5: footprint (none) -> Library:StandardUnpolarizedCapacitorPedal
- D2: footprint (none) -> Library:StandardDiode1N4000
- Q1: footprint MMBF5457_:SOT23 -> Library:SOT23
- R1, R10, R11, R12, R13, R14, R15, R16, R2, R3, R4, R5, R6, R7, R8, R9: footprint (none) -> Library:StandardResistorPedal
- RV1: footprint (none) -> Library:StandardPot
- SW1: footprint (none) -> Button_Switch_THT:SW_DIP_SPSTx02_Slide_6.7x6.64mm_W7.62mm_P2.54mm_LowProfile
Connections:
- net +9V: now also H7.1
- net Earth: now also H4.1, H5.1, H6.1, H8.1
- net SWA1: now also SW1.4; no longer SW1.1
- net SWA2: now also SW1.1; no longer SW1.4
- net IN: no longer names the net of C3.1, R5.1
- net IN: now also H2.1
- net OUT renamed SWB2
- net SWB2: now also H3.1
- net SW.: no longer names the net of D2.1 (K)
- net SW.: now also H1.1
Other:
- moved on the sheet: D2, SW1

Commit message: V2.0
Parts:
- added H10, H11, H12, H9: MountingHole_Pad, MountingHole:MountingHole_2.2mm_M2_DIN965_Pad, symbol Mechanical:MountingHole_Pad
- C5: value 33n -> 10u
- R14: value 100R -> 100
- R2: value 390R -> 390
Connections:
- net Earth: now also H10.1, H11.1, H12.1, H9.1
